Commit message: Fixed URDF for RViz2 display, except for colors

File: rccar_ws/src/rccar_lab/description/robot_core.xacro (robot description, xacro)
@@ -4,5 +4,33 @@
      For more information, please see http://wiki.ros.org/sw_urdf_exporter -->
 <robot
+  xmlns:xacro="http://www.ros.org/wiki/xacro"
   name="robot">
+  <!-- Material Definitions -->
+  <material
+    name="chassis_color">
+    <color
+      rgba="0.752941176470588 0.752941176470588 0.752941176470588 1" />
+  </material>
+  <material
+    name="ebox_color">
+    <color
+      rgba="0 0 0 1" />
+  </material>
+  <material
+    name="battery_color">
+    <color
+      rgba="0.250980392156863 0.250980392156863 0.250980392156863 1" />
+  </material>
+  <material
+    name="lidar_color">
+    <color
+      rgba="0.792156862745098 0.819607843137255 0.933333333333333 1" />
+  </material>
+  <material
+    name="wheel_color">
+    <color
+      rgba="0.792156862745098 0.819607843137255 0.933333333333333 1" />
+  </material>
+  <!-- Robot -->
   <link
     name="base_link">
@@ -33,8 +61,5 @@
       </geometry>
       <material
-        name="">
-        <color
-          rgba="0.752941176470588 0.752941176470588 0.752941176470588 1" />
-      </material>
+        name="chassis_color"/>
     </visual>
     <collision>
@@ -86,8 +111,5 @@
       </geometry>
       <material
-        name="">
-        <color
-          rgba="0 0 0 1" />
-      </material>
+        name="ebox_color"/>
     </visual>
     <collision>
@@ -106,5 +128,5 @@
     <origin
       xyz="-0.0036768 -0.095982 0.0485"
-      rpy="0 0 0" />
+      rpy="${pi/2} 0 0" />
     <parent
       link="chassis_link" />
@@ -139,8 +161,5 @@
       </geometry>
       <material
-        name="">
-        <color
-          rgba="0.250980392156863 0.250980392156863 0.250980392156863 1" />
-      </material>
+        name="battery_color"/>
     </visual>
     <collision>
@@ -159,5 +178,5 @@
     <origin
       xyz="-0.0036768 -0.095982 0.0285"
-      rpy="0 0 0" />
+      rpy="${pi/2} 0 0" />
     <parent
       link="chassis_link" />
@@ -192,8 +211,5 @@
       </geometry>
       <material
-        name="">
-        <color
-          rgba="0.792156862745098 0.819607843137255 0.933333333333333 1" />
-      </material>
+        name="lidar_color"/>
     </visual>
     <collision>
@@ -212,5 +228,5 @@
     <origin
       xyz="-0.016177 -0.095982 0.13493"
-      rpy="0 0 0" />
+      rpy="${pi/2} 0 0" />
     <parent
       link="chassis_link" />
@@ -245,8 +261,5 @@
       </geometry>
       <material
-        name="wheel_color">
-        <color
-          rgba="0.792156862745098 0.819607843137255 0.933333333333333 1" />
-      </material>
+        name="wheel_color"/>
     </visual>
     <collision>
@@ -298,8 +311,5 @@
       </geometry>
       <material
-        name="">
-        <color
-          rgba="0.792156862745098 0.819607843137255 0.933333333333333 1" />
-      </material>
+        name="wheel_color"/>
     </visual>
     <collision>
@@ -351,8 +361,5 @@
       </geometry>
       <material
-        name="">
-        <color
-          rgba="0.792156862745098 0.819607843137255 0.933333333333333 1" />
-      </material>
+        name="wheel_color"/>
     </visual>
     <collision>
@@ -404,8 +411,5 @@
       </geometry>
       <material
-        name="">
-        <color
-          rgba="0.792156862745098 0.819607843137255 0.933333333333333 1" />
-      </material>
+        name="wheel_color"/>
     </visual>
     <collision>

Commit message: Updated gazebo color tags

File: rccar_ws/src/rccar_lab/description/robot_core.xacro (robot description, xacro)
@@ -36,4 +36,5 @@
     name="base_link">
   </link>
+  <!-- Chassis -->
   <link
     name="chassis_link">
@@ -86,4 +87,8 @@
       xyz="0 0 0" />
   </joint>
+  <gazebo reference="chassis_link">
+      <material>Gazebo/Grey</material>
+  </gazebo>
+  <!-- Electrical Box -->
   <link
     name="ebox_link">
@@ -136,4 +141,8 @@
       xyz="0 0 0" />
   </joint>
+  <gazebo reference="ebox_link">
+    <material>Gazebo/DarkGrey</material>
+  </gazebo>
+  <!-- Battery -->
   <link
     name="battery_link">
@@ -186,4 +195,8 @@
       xyz="0 0 0" />
   </joint>
+    <gazebo reference="battery_link">
+      <material>Gazebo/DarkGrey</material>
+  </gazebo>
+  <!-- LiDAR -->
   <link
     name="lidar_link">
@@ -236,4 +249,8 @@
       xyz="0 0 0" />
   </joint>
+  <gazebo reference="lidar_link">
+      <material>Gazebo/DarkGrey</material>
+  </gazebo>
+  <!-- Front Right Wheel -->
   <link
     name="fr_wheel_link">
@@ -286,4 +303,8 @@
       xyz="0 1 0" />
   </joint>
+  <gazebo reference="fr_wheel_link">
+    <material>Gazebo/FlatBlack</material>
+  </gazebo>
+  <!-- Front Left Wheel -->
   <link
     name="fl_wheel_link">
@@ -336,4 +357,8 @@
       xyz="0 1 0" />
   </joint>
+  <gazebo reference="fr_wheel_link">
+    <material>Gazebo/FlatBlack</material>
+  </gazebo>
+  <!-- Back Left Wheel-->
   <link
     name="bl_wheel_link">
@@ -386,4 +411,8 @@
       xyz="0 1 0" />
   </joint>
+  <gazebo reference="bl_wheel_link">
+    <material>Gazebo/FlatBlack</material>
+  </gazebo>
+  <!-- Back Right Wheel -->
   <link
     name="br_wheel_link">
@@ -436,3 +465,6 @@
       xyz="0 1 0" />
   </joint>
+  <gazebo reference="br_wheel_link">
+    <material>Gazebo/FlatBlack</material>
+  </gazebo>
 </robot>
