Commit message: Figuring out Nav2, figured out SLAM

File: rccar_ws/src/rccar_lab/description/robot_core.xacro (robot description, xacro)
@@ -6,7 +6,17 @@
   xmlns:xacro="http://www.ros.org/wiki/xacro"
   name="robot">
+  <!-- BASE LINK -->
   <link
     name="base_link">
   </link>
+  <!-- BASE_FOOTPRINT LINK -->
+  <link name="base_footprint">
+  </link>
+  <joint name="base_footprint_joint" type="fixed">
+    <parent link="base_link"/>
+    <child link="base_footprint"/>
+    <origin xyz="0 0 0" rpy="0 0 0"/>
+  </joint>
+  <!-- CHASSIS LINK -->
   <link
     name="chassis_link">
