Commit message: Simulation now works with actual robot design

File: rccar_ws/src/rccar_lab/description/robot.urdf.xacro (robot description, xacro)
@@ -1,5 +1,5 @@
 <?xml version="1.0"?>
 <robot xmlns:xacro="http://www.ros.org/wiki/xacro" name = "robot">
-    <xacro:include filename="test_robot.xacro"/>
-    <xacro:include filename="test_control.xacro"/>
+    <xacro:include filename="robot_core.xacro"/>
+    <xacro:include filename="ros2_control.xacro"/>
 </robot>

File: rccar_ws/src/rccar_lab/description/ros2_control.xacro (robot description, xacro)
@@ -8,18 +8,17 @@
         </hardware>
         <!-- Now specify the joints it will be controlling based on robot URDF -->
-        <joint name="fr_wheel_joint">
+        <joint name="fl_wheel_joint">
             <!-- Current values are arbitrary -->
             <command_interface name="velocity">
-                <param name="min">-10</param>
-                <param name="max">10</param>
+                <param name="min">-40</param>
+                <param name="max">40</param>
             </command_interface>
             <state_interface name="velocity"/>
             <state_interface name="position"/>
         </joint>
-        <joint name="fl_wheel_joint">
-            <!-- Current values are arbitrary -->
+        <joint name="fr_wheel_joint">
             <command_interface name="velocity">
-                <param name="min">-10</param>
-                <param name="max">10</param>
+                <param name="min">-40</param>
+                <param name="max">40</param>
             </command_interface>
             <state_interface name="velocity"/>
@@ -27,8 +26,7 @@
         </joint>
         <joint name="br_wheel_joint">
-            <!-- Current values are arbitrary -->
             <command_interface name="velocity">
-                <param name="min">-10</param>
-                <param name="max">10</param>
+                <param name="min">-40</param>
+                <param name="max">40</param>
             </command_interface>
             <state_interface name="velocity"/>
@@ -36,8 +34,7 @@
         </joint>
         <joint name="bl_wheel_joint">
-            <!-- Current values are arbitrary -->
             <command_interface name="velocity">
-                <param name="min">-10</param>
-                <param name="max">10</param>
+                <param name="min">-40</param>
+                <param name="max">40</param>
             </command_interface>
             <state_interface name="velocity"/>
@@ -49,5 +46,5 @@
     <gazebo>
         <plugin
-        filename="gz_ros2_control-system"
+        filename="libgz_ros2_control-system.so"
         name="gz_ros2_control::GazeboSimROS2ControlPlugin"
         >
