Commit message: Fixed Gazebo motion by setting all wheels to rotate around xyz = 0 1 0

File: rccar_ws/src/rccar_lab/car_urdf/urdf/car_urdf.urdf (robot description, URDF)
Before this commit: robot robot, 9 links, 8 joints
Links:
- link chassis_link: mass 0.0660834014682612 -> 0.253438557114572
Joints:
- joint bl_wheel_joint: axis 0 1 0 -> 0 -1 0; origin xyz=0.0549999999999999 -0.0383500000000002 -0.0134999999999998 rpy=0 0 0 -> xyz=-0.055 0.05545 -0.0135 rpy=0 0 0
- joint br_wheel_joint: axis 0 -1 0 -> 0 1 0; origin xyz=0.0550000000000002 0.0383499999999998 -0.0134999999999998 rpy=0 0 0 -> xyz=-0.055 -0.05545 -0.0135 rpy=0 0 0
- joint ebox_joint: origin xyz=0 0 0.00249999999999995 rpy=0 0 0 -> xyz=0 0 0.0025 rpy=0 0 0
- joint fl_wheel_joint: axis 0 1 0 -> 0 -1 0; origin xyz=-0.0550000000000001 -0.0403499999999998 -0.0135000000000002 rpy=0 0 0 -> xyz=0.055 0.05745 -0.0135 rpy=0 0 0
- joint fr_wheel_joint: axis 0 -1 0 -> 0 1 0; origin xyz=-0.0549999999999998 0.0383500000000002 -0.0135000000000002 rpy=0 0 0 -> xyz=0.055 -0.05545 -0.0135 rpy=0 0 0
- joint laser_frame_joint: origin xyz=0 -0.0124999669534474 0.0889299999999999 rpy=0 0 0 -> xyz=0 0.0125 0.08893 rpy=0 0 0

File: rccar_ws/src/rccar_lab/description/robot_core.xacro (robot description, xacro)
@@ -13,15 +13,15 @@
     <inertial>
       <origin
-        xyz="-1.50742878161203E-16 -4.16333634234428E-17 0.0349999999999999"
-        rpy="0 0 0" />
-      <mass
-        value="0.0660834014682612" />
-      <inertia
-        ixx="6.99540118235905E-05"
-        ixy="2.06199956920822E-22"
-        ixz="-2.43487880406245E-19"
-        iyy="7.00130698384872E-05"
-        iyz="8.50154197152472E-34"
-        izz="0.00013969173415596" />
+        xyz="0.000204687581195852 0.00314875501574724 1.53572466782085E-17"
+        rpy="0 0 0" />
+      <mass
+        value="0.253438557114572" />
+      <inertia
+        ixx="0.000230915983626971"
+        ixy="-1.25922435715914E-21"
+        ixz="-1.96530082780382E-20"
+        iyy="0.000388552862570868"
+        iyz="8.63727389926082E-21"
+        izz="0.000171792964937591" />
     </inertial>
     <visual>
@@ -36,5 +36,5 @@
         name="">
         <color
-          rgba="0.250980392156863 0.250980392156863 0.250980392156863 1" />
+          rgba="0.752941176470588 0.752941176470588 0.752941176470588 1" />
       </material>
     </visual>
@@ -66,5 +66,5 @@
     <inertial>
       <origin
-        xyz="9.71445146547012E-17 0.0170468370852515 -2.42861286636753E-17"
+        xyz="6.93889390390723E-18 5.31629147485363E-05 1.04083408558608E-17"
         rpy="0 0 0" />
       <mass
@@ -72,8 +72,8 @@
       <inertia
         ixx="2.49513056185901E-05"
-        ixy="6.59448174057087E-20"
-        ixz="-3.87740912134232E-22"
+        ixy="-5.423278565198E-20"
+        ixz="4.13590306276502E-22"
         iyy="4.21618272671167E-05"
-        iyz="1.03511386444233E-22"
+        iyz="-9.47970035310487E-23"
         izz="2.49513056185901E-05" />
     </inertial>
@@ -106,5 +106,5 @@
     type="continuous">
     <origin
-      xyz="-0.0549999999999998 0.0383500000000002 -0.0135000000000002"
+      xyz="0.055 -0.05545 -0.0135"
       rpy="0 0 0" />
     <parent
@@ -113,5 +113,5 @@
       link="fr_wheel_link" />
     <axis
-      xyz="0 -1 0" />
+      xyz="0 1 0" />
   </joint>
   <link
@@ -119,5 +119,5 @@
     <inertial>
       <origin
-        xyz="-3.46944695195361E-17 -0.0170468370852515 -4.68375338513738E-17"
+        xyz="0 -5.31629147485432E-05 -5.20417042793042E-18"
         rpy="0 0 0" />
       <mass
@@ -125,8 +125,8 @@
       <inertia
         ixx="2.49513056185901E-05"
-        ixy="6.54299744512327E-20"
-        ixz="2.64956289958392E-22"
+        ixy="-5.47674516841756E-20"
+        ixz="-2.71418638493962E-22"
         iyy="4.21618272671167E-05"
-        iyz="-2.13911019413315E-22"
+        iyz="2.30183165982362E-22"
         izz="2.49513056185901E-05" />
     </inertial>
@@ -159,5 +159,5 @@
     type="continuous">
     <origin
-      xyz="-0.0550000000000001 -0.0403499999999998 -0.0135000000000002"
+      xyz="0.055 0.05745 -0.0135"
       rpy="0 0 0" />
     <parent
@@ -172,5 +172,5 @@
     <inertial>
       <origin
-        xyz="6.24500451351651E-17 0.0170468370852515 -3.29597460435593E-17"
+        xyz="0 5.31629147485363E-05 1.73472347597681E-18"
         rpy="0 0 0" />
       <mass
@@ -178,8 +178,8 @@
       <inertia
         ixx="2.49513056185901E-05"
-        ixy="5.51824614792902E-20"
-        ixz="-6.87836222254764E-22"
+        ixy="-6.50129727077473E-20"
+        ixz="6.75315421967096E-22"
         iyy="4.21618272671167E-05"
-        iyz="-1.18907017039843E-21"
+        iyz="1.17926037236496E-21"
         izz="2.49513056185901E-05" />
     </inertial>
@@ -212,5 +212,5 @@
     type="continuous">
     <origin
-      xyz="0.0550000000000002 0.0383499999999998 -0.0134999999999998"
+      xyz="-0.055 -0.05545 -0.0135"
       rpy="0 0 0" />
     <parent
@@ -219,5 +219,5 @@
       link="br_wheel_link" />
     <axis
-      xyz="0 -1 0" />
+      xyz="0 1 0" />
   </joint>
   <link
@@ -225,5 +225,5 @@
     <inertial>
       <origin
-        xyz="-2.77555756156289E-17 -0.0170468370852515 -3.64291929955129E-17"
+        xyz="-6.93889390390723E-18 -5.31629147485502E-05 -1.73472347597681E-18"
         rpy="0 0 0" />
       <mass
@@ -231,8 +231,8 @@
       <inertia
         ixx="2.49513056185901E-05"
-        ixy="6.33951344235919E-20"
-        ixz="1.78522378295136E-21"
+        ixy="-5.67907179160895E-20"
+        ixz="-1.78845495721914E-21"
         iyy="4.21618272671167E-05"
-        iyz="-9.05830818008876E-22"
+        iyz="9.13026509813255E-22"
         izz="2.49513056185901E-05" />
     </inertial>
@@ -265,5 +265,5 @@
     type="continuous">
     <origin
-      xyz="0.0549999999999999 -0.0383500000000002 -0.0134999999999998"
+      xyz="-0.055 0.05545 -0.0135"
       rpy="0 0 0" />
     <parent
@@ -278,5 +278,5 @@
     <inertial>
       <origin
-        xyz="1.57173789229634E-16 0.00645097632173484 -0.0220370930302957"
+        xyz="-1.11844852964053E-16 -0.00645097632173484 -0.0220370930302957"
         rpy="0 0 0" />
       <mass
@@ -284,8 +284,8 @@
       <inertia
         ixx="0.0002404496804147"
-        ixy="-3.1288892395143E-19"
-        ixz="1.32912845998458E-19"
+        ixy="1.12972461375983E-19"
+        ixz="-7.32140473318081E-21"
         iyy="0.000179322343491855"
-        iyz="1.7915823262772E-05"
+        iyz="-1.7915823262772E-05"
         izz="0.00023562662350046" />
     </inertial>
@@ -318,5 +318,5 @@
     type="fixed">
     <origin
-      xyz="0 -0.0124999669534474 0.0889299999999999"
+      xyz="0 0.0125 0.08893"
       rpy="0 0 0" />
     <parent
@@ -363,5 +363,5 @@
     <inertial>
       <origin
-        xyz="-2.34699262998591E-18 7.10678486645065E-18 0.00665420516682762"
+        xyz="1.32591217148186E-18 -7.42445710199543E-18 0.00665420516682762"
         rpy="0 0 0" />
       <mass
@@ -369,8 +369,8 @@
       <inertia
         ixx="1.44863163441746E-05"
-        ixy="-3.28171735040022E-20"
-        ixz="-1.68952862307112E-20"
+        ixy="2.72159329107965E-20"
+        ixz="1.70283301056841E-20"
         iyy="5.88923381835338E-06"
-        iyz="-7.36044596547253E-22"
+        iyz="8.0720709024853E-22"
         izz="1.88651943786396E-05" />
     </inertial>
@@ -403,5 +403,5 @@
     type="fixed">
     <origin
-      xyz="0 0 0.00249999999999995"
+      xyz="0 0 0.0025"
       rpy="0 0 0" />
     <parent
@@ -416,5 +416,5 @@
     <inertial>
       <origin
-        xyz="0.000123841648641815 -5.16561475905226E-18 0.00748048339939821"
+        xyz="-0.000123841648641815 4.21830740490866E-18 0.00748048339939821"
         rpy="0 0 0" />
       <mass
@@ -422,8 +422,8 @@
       <inertia
         ixx="2.44479179923402E-06"
-        ixy="2.77230971591075E-20"
-        ixz="-6.80855024106344E-11"
+        ixy="-2.98803775987149E-20"
+        ixz="6.80855024106424E-11"
         iyy="1.06924152126357E-05"
-        iyz="2.21389541828885E-23"
+        iyz="-2.10030338456889E-23"
         izz="1.21105909928422E-05" />
     </inertial>
